File: MPF-III/Keyboard/MPF-III_Keyboard/MPF-III_Keyboard.kicad_sch (KiCad schematic)
At the start: 2 parts, among them J1 MPF-III U78, J2 MPF-III Keyboard Socket

Commit message: Initial commit
Connections:
- net CLOCK renamed KB_CLK
- net DATA renamed KB_DATA
Changed lines of the file:
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@@
 		)
 	)
-	(text_box "PB0: If you want to invoke a cold-start, you may first press [CTRL] and [RESET] simultaneously, followed by a press on PB0 and then yuou release [CTRL] and [RESET] followed by [PB0]. In so doing you can do without powering off the system.\n\nPB1: This key is used for self-test of the system. First, Press [CTRL] [RESET], followed by pressing [PB1]. Release [CTRL] [RESET] first and then [PB1].  After these steps are completed, the MPF-III will stasrt testing RAM, ROM, together with SG and Colour Bar Test.\n"
+	(text_box "PB0: If you want to invoke a cold-start, you may first press [CTRL] and [RESET] simultaneously, followed by a press on PB0 and then yuou release [CTRL] and [RESET] followed by [PB0]. In so doing you can do without powering off the system.\n\nPB1: This key is used for self-test of the system. First, press [CTRL] [RESET], followed by pressing [PB1]. Release [CTRL] [RESET] first and then [PB1].  After these steps are completed, the MPF-III will start testing RAM, ROM, together with Sound Generator and Colour Bar Test.\n\nAKD: Any Key Down.  If any key is pressed, the signal is high.  Otherwise, it is low.\n"
 		(exclude_from_sim no)
 		(at 172.72 59.69 0)
@@
 		)
 	)
-	(global_label "DATA"
+	(global_label "KB_DATA"
 		(shape input)
 		(at 113.03 82.55 180)
@@
 		)
 		(property "Intersheetrefs" "${INTERSHEET_REFS}"
-			(at 105.63 82.55 0)
+			(at 102.1224 82.55 0)
 			(effects
 				(font
@@
 		)
 	)
-	(global_label "CLOCK"
+	(global_label "KB_CLK"
 		(shape input)
 		(at 113.03 77.47 180)
@@
 		)
 		(property "Intersheetrefs" "${INTERSHEET_REFS}"
-			(at 103.8762 77.47 0)
+			(at 102.9691 77.47 0)
 			(effects
 				(font
