File: MPF-III/Keyboard/MPF-III_Keyboard/MPF-III_Keyboard.kicad_sch (KiCad schematic)
At the start: 96 parts, among them J1 MPF-III U78, J2 MPF-III Keyboard Socket, SW1 F1, SW10 F10, SW11 F11, SW12 F12, SW13 PB0, SW14 PB1, SW15 BREAK, SW16 RESET, SW17 NUM LOCK, SW18 HALT, SW19 ESC, SW2 F2, SW20 ! 1, SW21 @ 2, SW22 # 3, SW23 $ 4, SW24 % 5, SW25 ^ 6, SW26 & 7, SW27 * 8, SW28 ( 9, SW29 ) 0, SW3 F3, SW30 _ -, SW31 + =, SW32 <--, SW33 TAB, SW34 Q, SW35 W, SW36 E, SW37 R, SW38 T, SW39 Y, SW4 F4, SW40 U, SW41 I, SW42 O, SW43 P, SW44 { [, SW45 } ], SW46 DEL, SW47 NP 7, SW48 NP 8, SW49 NP 9, SW5 F5, SW50 NP -, SW51 NP 4, SW52 NP 5, SW53 NP 6, SW54 NP +, SW55 CTRL, SW56 A, SW57 S, SW58 D, SW59 F, SW6 F6, SW60 G, SW61 H, SW62 J, SW63 K, SW64 L, SW65 : ;, SW66 " ', SW67 ~ `, SW68 RETURN, SW69 NP 1, SW7 F7, SW70 NP 2, SW71 NP 3, SW72 NP RETURN, SW73 LH SHIFT, SW74 | \, SW75 Z, SW76 X, SW77 C, SW78 V, SW79 B, SW8 F8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

Commit message: Started PCB layout
Parts:
- added H1, H2, H3, H4, H5, H6: MountingHole, MountingHole:MountingHole_3.2mm_M3, symbol Mechanical:MountingHole
Other:
- moved on the sheet: SW55, SW73, SW85, SW86
